File: KiCAD/e-cribbage.kicad_pcb (KiCad board)
At the start: 2 copper layers, 269.7 x 100.3 mm, 559 parts, among them U1 74HC595D_118, U10 74HC595D_118, U11 74HC595D_118, U12 74HC595D_118, U13 74HC595D_118, U14 74HC595D_118, U15 74HC595D_118, U16 74HC595D_118, U17 74HC595D_118, U18 74HC595D_118, U19 74HC595D_118, U2 MSP430F2012IPW, U20 74HC595D_118, U21 74HC595D_118, U22 74HC595D_118, U23 74HC595D_118, U24 74HC595D_118, U25 74HC595D_118, U26 74HC595D_118, U27 74HC595D_118, U28 74HC595D_118, U29 74HC595D_118, U3 74HC595D_118, U30 74HC595D_118, U31 74HC595D_118, U32 SN74LVC1G08DBVR, U33 SN74LVC1G125DCKR, U4 74HC595D_118, U5 74HC595D_118, U6 74HC595D_118, U7 74HC595D_118, U8 74HC595D_118, U9 74HC595D_118

Commit message: reduced 0603 footprints
Parts:
- D100, D101, D102, D103, D104, D105, D106, D107, D108, D109, D11, D110, D111, D112, D113, D114, D115, D116, D117, D118, D119, D12, D120, D121, D122, D123, D124, D125, D126, D127, D128, D129, D13, D130, D131, D132, D133, D134, D135, D136, D137, D138, D139, D14, D140, D141, D142, D143, D144, D145, D146, D147, D148, D149, D15, D150, D151, D152, D153, D154, D155, D156, D157, D158, D159, D16, D160, D161, D162, D163, D164, D165, D166, D167, D168, D169, D17, D170, D171, D172, D173, D174, D175, D176, D177, D178, D179, D18, D180, D181, D182, D183, D184, D185, D186, D187, D188, D189, D19, D190, D191, D192, D193, D194, D195, D196, D197, D198, D199, D20, D200, D201, D202, D203, D204, D205, D206, D207, D208, D209, D21, D210, D211, D212, D213, D214, D215, D216, D217, D218, D219, D22, D220, D221, D222, D223, D224, D225, D226, D227, D228, D229, D23, D230, D231, D232, D233, D234, D235, D236, D237, D238, D239, D24, D240, D25, D26, D27, D28, D29, D30, D31, D32, D33, D34, D35, D36, D37, D38, D39, D40, D41, D42, D43, D44, D45, D46, D47, D48, D49, D50, D51, D52, D53, D54, D55, D56, D57, D58, D59, D60, D61, D62, D63, D64, D65, D66, D67, D68, D69, D70, D71, D72, D73, D74, D75, D76, D77, D78, D79, D80, D81, D82, D83, D84, D85, D86, D87, D88, D89, D90, D91, D92, D93, D94, D95, D96, D97, D98, D99: footprint LEDs:LED_0603_HandSoldering -> LEDs:LED_0603
- R100, R101, R102, R103, R104, R105, R106, R107, R108, R109, R11, R110, R111, R112, R113, R114, R115, R116, R117, R118, R119, R12, R120, R121, R122, R123, R124, R125, R126, R127, R128, R129, R13, R130, R131, R132, R133, R134, R135, R136, R137, R138, R139, R14, R140, R141, R142, R143, R144, R145, R146, R147, R148, R149, R15, R150, R151, R152, R153, R154, R155, R156, R157, R158, R159, R16, R160, R161, R162, R163, R164, R165, R166, R167, R168, R169, R17, R170, R171, R172, R173, R174, R175, R176, R177, R178, R179, R18, R180, R181, R182, R183, R184, R185, R186, R187, R188, R189, R19, R190, R191, R192, R193, R194, R195, R196, R197, R198, R199, R20, R200, R201, R202, R203, R204, R205, R206, R207, R208, R209, R21, R210, R211, R212, R213, R214, R215, R216, R217, R218, R219, R22, R220, R221, R222, R223, R224, R225, R226, R227, R228, R229, R23, R230, R231, R232, R233, R234, R235, R236, R237, R238, R239, R24, R240, R241, R242, R243, R244, R245, R246, R247, R248, R249, R25, R250, R26, R27, R28, R29, R30, R31, R32, R33, R34, R35, R36, R37, R38, R39, R40, R41, R42, R43, R44, R45, R46, R47, R48, R49, R50, R51, R52, R53, R54, R55, R56, R57, R58, R59, R60, R61, R62, R63, R64, R65, R66, R67, R68, R69, R70, R71, R72, R73, R74, R75, R76, R77, R78, R79, R80, R81, R82, R83, R84, R85, R86, R87, R88, R89, R90, R91, R92, R93, R94, R95, R96, R97, R98, R99: footprint Resistors_SMD:R_0603_HandSoldering -> Resistors_SMD:R_0603
- moved C22 38.4 mm to (135.1, 114.0)
- moved C15 13.2 mm to (122.2, 118.5)
- moved C21 13.2 mm to (128.4, 114.0)
- moved C23 13.2 mm to (133.9, 104.3)
- moved C25 13.2 mm to (128.4, 109.3)
- moved C28 13.2 mm to (128.4, 111.7)
- moved C30 13.2 mm to (133.9, 101.9)
- moved C8 13.2 mm to (133.3, 96.3)
- moved C10 13.2 mm to (122.2, 116.1)
- moved C24 13.2 mm to (128.6, 106.0)
- moved C27 13.2 mm to (128.9, 101.3)
- moved C29 13.2 mm to (122.8, 110.2)
- moved C31 13.2 mm to (122.8, 107.8)
- moved C26 13.2 mm to (132.9, 107.4)
Routing:
- net GND: track 201.8 -> 206.9 mm
- net Net-(D129-Pad2): track 63.9 -> 65.7 mm
- net +3V3: track 95.5 -> 96.7 mm, vias 8 -> 9

Commit message: power and ground planes added 471 nets unconnected
Parts:
- added C32: 1.0uF, Capacitors_SMD:C_0603_HandSoldering, F.Cu at (89.7, 228.5)
- added C33: 1.0uF, Capacitors_SMD:C_0603_HandSoldering, F.Cu at (89.7, 230.9)
- added C34: 1.0uF, Capacitors_SMD:C_0603_HandSoldering, F.Cu at (94.4, 228.5)
- added C35: 1.0uF, Capacitors_SMD:C_0603_HandSoldering, F.Cu at (89.7, 233.2)
- added R251: 47k, Resistors_SMD:R_0603, F.Cu at (93.8, 230.9)
- moved C14 122.3 mm to (21.1, 184.7)
- moved U14 109.2 mm to (261.9, 183.1), turned to 270 degrees
- moved U27 102.4 mm to (110.0, 183.4)
- moved U22 100.1 mm to (243.8, 158.0), turned to 270 degrees
- moved U26 99.1 mm to (93.0, 183.9), turned to 90 degrees
- moved U23 98.3 mm to (182.9, 157.7), turned to 270 degrees
- moved R241 92.9 mm to (40.4, 130.3), turned to 180 degrees
- moved U12 86.8 mm to (143.3, 183.1), turned to 270 degrees
- moved U13 83.8 mm to (160.3, 183.4)
- moved U10 73.7 mm to (86.6, 158.0)
- moved U21 67.5 mm to (281.9, 132.8), turned to 0 degrees
- moved U25 64.2 mm to (57.9, 158.0)
- moved U15 63.1 mm to (288.0, 201.7), turned to 270 degrees
- moved U28 58.7 mm to (195.8, 183.9), turned to 90 degrees
- moved U11 54.1 mm to (74.7, 183.4)
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Connections:
- R243 pad 1: (no net) -> Net-(C32-Pad1)
- R243 pad 2: (no net) -> +3V3
- R244 pad 1: (no net) -> Net-(C35-Pad1)
- R244 pad 2: (no net) -> +3V3
- R246 pad 1: (no net) -> Net-(C34-Pad1)
- R246 pad 2: (no net) -> +3V3
- R247 pad 1: (no net) -> Net-(C33-Pad1)
- R247 pad 2: (no net) -> +3V3
- S1 pad 1: Net-(S1-Pad1) -> Net-(C32-Pad1)
- S1 pad 2: Net-(S1-Pad2) -> GND
- S2 pad 1: Net-(S2-Pad1) -> Net-(C33-Pad1)
- S2 pad 2: Net-(S2-Pad2) -> GND
- S3 pad 1: Net-(S3-Pad1) -> Net-(C34-Pad1)
- S3 pad 2: Net-(S3-Pad2) -> GND
- S4 pad 1: Net-(S4-Pad1) -> Net-(C35-Pad1)
- S4 pad 2: Net-(S4-Pad2) -> GND
- U2 pad 10: (no net) -> RST
- U2 pad 2: (no net) -> Net-(C32-Pad1)
- U2 pad 3: (no net) -> Net-(C33-Pad1)
- U2 pad 4: (no net) -> Net-(C34-Pad1)
- U2 pad 5: (no net) -> Net-(C35-Pad1)
Routing:
- net GND: track 206.9 -> 395.8 mm, vias 56 -> 225
- net Net-(R241-Pad1): track 0.00 -> 8.29 mm
- net +3V3: track 96.7 -> 101.4 mm
- net Net-(D69-Pad1): track 2.96 -> 0.00 mm
- net Net-(D70-Pad1): track 3.13 -> 0.25 mm
- net Net-(D68-Pad1): track 2.96 -> 0.08 mm
- net Net-(D67-Pad1): track 3.13 -> 0.25 mm
- net Net-(D66-Pad1): track 2.96 -> 0.08 mm
- net Net-(D65-Pad1): track 3.13 -> 0.25 mm
- net Net-(D64-Pad1): track 2.96 -> 0.08 mm
- net Net-(D63-Pad1): track 3.04 -> 0.17 mm
- net Net-(D62-Pad1): track 2.96 -> 0.08 mm
- net Net-(D24-Pad1): track 2.96 -> 0.08 mm
- net Net-(D23-Pad1): track 2.87 -> 0.00 mm
- net Net-(D178-Pad1): track 0.00 -> 2.79 mm
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
Commit message: preliminary part placement and route
Parts:
- removed R241, R242, R245, R248, R249, R250: 10k, Resistors_SMD:R_0603
- removed U33: SN74LVC1G125DCKR, digikey-footprints:SOT-353
- added C36: 1.0uF, Capacitors_SMD:C_0603_HandSoldering, F.Cu at (119.9, 198.5)
- added C37: 1.0uF, Capacitors_SMD:C_0603_HandSoldering, F.Cu at (124.6, 198.5)
- added C38: 1.0uF, Capacitors_SMD:C_0603_HandSoldering, F.Cu at (129.2, 198.5)
- added C39: 1.0uF, Capacitors_SMD:C_0603_HandSoldering, F.Cu at (138.7, 187.9)
- added U34: SN74LVC1G08DBVR, digikey-footprints:SOT-753, F.Cu at (197.4, 163.6)
- added U35: SN74LVC1G08DBVR, digikey-footprints:SOT-753, F.Cu at (204.7, 163.6)
- added U36: SN74LVC1G08DBVR, digikey-footprints:SOT-753, F.Cu at (214.1, 163.6)
- added U37: SN74LVC1G08DBVR, digikey-footprints:SOT-753, F.Cu at (221.5, 163.6)
- added U38: SN74LVC1G08DBVR, digikey-footprints:SOT-753, F.Cu at (228.8, 163.6)
- added U39: SN74LVC1G08DBVR, digikey-footprints:SOT-753, F.Cu at (236.7, 163.6)
- added U40: SN74LVC1G08DBVR, digikey-footprints:SOT-753, F.Cu at (243.3, 163.6)
- moved C14 308.3 mm to (326.4, 141.7), turned to 90 degrees
- moved C15 230.3 mm to (347.7, 165.1), turned to 90 degrees
- moved C21 220.5 mm to (348.2, 96.8), turned to 270 degrees
- moved C13 213.1 mm to (226.0, 155.2), turned to 0 degrees
- moved C30 203.4 mm to (333.5, 141.2), turned to 90 degrees
- moved C12 190.2 mm to (208.5, 141.0), turned to 0 degrees
- moved C22 155.0 mm to (290.1, 116.6)
- moved C29 152.4 mm to (271.5, 143.5), turned to 270 degrees
- moved C31 152.1 mm to (263.4, 166.1), turned to 90 degrees
- moved C8 145.4 mm to (277.4, 115.6)
- moved C28 118.2 mm to (242.1, 143.8)
- moved S4 112.4 mm to (79.6, 153.2)
- moved S3 112.4 mm to (62.5, 153.2)
- moved U32 108.8 mm to (189.5, 163.6)
- moved S1 101.7 mm to (62.7, 124.2)
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Connections:
- U1 pad 10: Net-(R241-Pad1) -> +3V3
- U1 pad 11: CLK -> CLK1A
- U1 pad 12: CLK -> CLK1A
- U1 pad 13: Net-(R241-Pad1) -> +3V3
- U15 pad 10: (no net) -> +3V3
- U15 pad 13: (no net) -> +3V3
- U16 pad 10: (no net) -> +3V3
- U16 pad 13: (no net) -> +3V3
- U2 pad 12: (no net) -> LE2
- U2 pad 13: (no net) -> LE1
- U3 pad 10: Net-(R242-Pad1) -> +3V3
- U3 pad 11: (no net) -> CLK1A
- U3 pad 12: (no net) -> CLK1A
- U3 pad 13: Net-(R242-Pad1) -> +3V3
- U32 pad 1: (no net) -> LE1
- U32 pad 2: (no net) -> CLK
- U32 pad 3: (no net) -> GND
- U32 pad 4: (no net) -> CLK1A
- U32 pad 5: (no net) -> +3V3
- U4 pad 10: (no net) -> +3V3
- U4 pad 11: (no net) -> CLK1A
- U4 pad 12: (no net) -> CLK1A
- U4 pad 13: (no net) -> +3V3
- U5 pad 11: (no net) -> CLK1A
- U5 pad 12: (no net) -> CLK1A
Routing:
- net Net-(C33-Pad1): track 0.00 -> 209.7 mm, vias 0 -> 2
- net DATA: track 0.00 -> 201.8 mm, vias 0 -> 3
- net +3V3: track 101.4 -> 301.5 mm, vias 9 -> 53
- net GND: track 395.8 -> 594.2 mm, vias 225 -> 303
- net Net-(C35-Pad1): track 0.00 -> 187.0 mm, vias 0 -> 2
- net Net-(C32-Pad1): track 0.00 -> 182.5 mm, vias 0 -> 2
- net Net-(C34-Pad1): track 0.00 -> 168.4 mm, vias 0 -> 2
- net Net-(U30-Pad9): track 0.00 -> 161.3 mm, vias 0 -> 4
- net CLK: track 0.00 -> 141.6 mm
- net LE2: track 0.00 -> 101.1 mm, vias 0 -> 5
- net Net-(U21-Pad9): track 0.00 -> 97.2 mm, vias 0 -> 2
- net Net-(D232-Pad2): track 0.00 -> 82.8 mm, vias 0 -> 2
- net CLK1A: track 0.00 -> 81.3 mm, vias 0 -> 1
- net LE1: track 0.00 -> 77.9 mm, vias 0 -> 4
- net Net-(D194-Pad2): track 0.00 -> 75.9 mm, vias 0 -> 2
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Other:
- board size 269.7 x 100.3 mm -> 304.8 x 100.3 mm
- board text added: "FINISH"
- board text added: "PLAYER ONE START"
- board text added: "PLAYER TWO START"
